Commit message: Address Doug's first round of comments

File: motive_description/urdf/msa6_v03.urdf (robot description, URDF)
Before this commit: robot msa6, 8 links, 7 joints
Links:
- removed link link1
- removed link link2
- removed link link3
- removed link link4
- removed link link5
- removed link link6
- added link link_L1, mass 1000; collision mesh filename=package://motive_description/meshes/msa6/link_L0.STL; visual mesh filename=package://motive_description/meshes/msa6/link_L0.STL
- added link link_L2, mass 0.994568789062109; collision mesh filename=package://motive_description/meshes/msa6/link_L1.STL; visual mesh filename=package://motive_description/meshes/msa6/link_L1.STL
- added link link_L3, mass 1.03970207416395; collision mesh filename=package://motive_description/meshes/msa6/link_L2.STL; visual mesh filename=package://motive_description/meshes/msa6/link_L2.STL
- added link link_L4, mass 1.08371144697155; collision mesh filename=package://motive_description/meshes/msa6/link_L3.STL; visual mesh filename=package://motive_description/meshes/msa6/link_L3.STL
- added link link_L5, mass 1.06997840394961; collision mesh filename=package://motive_description/meshes/msa6/link_L4.STL; visual mesh filename=package://motive_description/meshes/msa6/link_L4.STL
- added link link_L6, mass 0.996094913930728; collision mesh filename=package://motive_description/meshes/msa6/link_L5.STL; visual mesh filename=package://motive_description/meshes/msa6/link_L5.STL
Joints:
- removed joint joint1
- removed joint joint2
- removed joint joint3
- removed joint joint4
- removed joint joint5
- removed joint joint6
- added joint joint_J1: type revolute, parent link_L1, child link_L2, origin xyz=0 0 0 rpy=0 0 -1.5708, axis 0 0 1, limit lower=-3 upper=3 effort=10 velocity=3
- added joint joint_J2: type revolute, parent link_L2, child link_L3, origin xyz=0.1 0 0.053637 rpy=0 1.5708 0, axis 0 0 1, limit lower=-3 upper=3 effort=10 velocity=3
- added joint joint_J3: type revolute, parent link_L3, child link_L4, origin xyz=-0.061373 0 0.1 rpy=3.1416 -1.5708 3.1416, axis 0 0 1, limit lower=-3 upper=3 effort=10 velocity=3
- added joint joint_J4: type revolute, parent link_L4, child link_L5, origin xyz=0.175 0 0.082746 rpy=0 0 0, axis 0 0 1, limit lower=-3 upper=3 effort=10 velocity=3
- added joint joint_J5: type revolute, parent link_L5, child link_L6, origin xyz=0.15 0 0 rpy=-3.1416 0 3.1416, axis 0 0 1, limit lower=-3 upper=3 effort=10 velocity=3
- added joint joint_J6: type revolute, parent link_L6, child link7, origin xyz=-0.09475 0 0.09475 rpy=-1.5708 -1.4987 1.5708, axis 0 0 1, limit lower=-3 upper=3 effort=10 velocity=3
- joint fixed: child link1 -> link_L1

Commit message: add msa6 meshes and update urdf

File: motive_description/urdf/msa6_v03.urdf (robot description, URDF)
Before this commit: robot msa6, 8 links, 7 joints
Links:
- removed link link7
- added link link_L0, mass 1.224; collision mesh filename=package://motive_description/meshes/msa6/link_L0.stl; visual mesh filename=package://motive_description/meshes/msa6/link_L0.stl
- link link_L1: mass 1000 -> 0.994568789062109; geometry collision mesh filename=package://motive_description/meshes/msa6/link_L1.stl; visual mesh filename=package://motive_description/meshes/msa6/link_L1.stl
- link link_L2: mass 0.994568789062109 -> 1.03970207416395; geometry collision mesh filename=package://motive_description/meshes/msa6/link_L2.stl; visual mesh filename=package://motive_description/meshes/msa6/link_L2.stl
- link link_L3: mass 1.03970207416395 -> 1.08371144697155; geometry collision mesh filename=package://motive_description/meshes/msa6/link_L3.stl; visual mesh filename=package://motive_description/meshes/msa6/link_L3.stl
- link link_L4: mass 1.08371144697155 -> 1.06997840394961; geometry collision mesh filename=package://motive_description/meshes/msa6/link_L4.stl; visual mesh filename=package://motive_description/meshes/msa6/link_L4.stl
- link link_L5: mass 1.06997840394961 -> 0.996094913930728; geometry collision mesh filename=package://motive_description/meshes/msa6/link_L5.stl; visual mesh filename=package://motive_description/meshes/msa6/link_L5.stl
- link link_L6: mass 0.996094913930728 -> 0.692011838300634; geometry collision mesh filename=package://motive_description/meshes/msa6/link_L6.stl; visual mesh filename=package://motive_description/meshes/msa6/link_L6.stl
Joints:
- joint fixed: child link_L1 -> link_L0; origin xyz=0 0 1 -> xyz=0 0 .15
- joint joint_J1: child link_L2 -> link_L1; limit lower=-3 upper=3 effort=10 velocity=3 -> lower=-2.74 upper=3.1 effort=14 velocity=3; parent link_L1 -> link_L0
- joint joint_J2: child link_L3 -> link_L2; limit lower=-3 upper=3 effort=10 velocity=3 -> lower=-2.92 upper=2.92 effort=14 velocity=3; parent link_L2 -> link_L1
- joint joint_J3: child link_L4 -> link_L3; limit lower=-3 upper=3 effort=10 velocity=3 -> lower=-3.28 upper=2.55 effort=14 velocity=6; parent link_L3 -> link_L2
- joint joint_J4: child link_L5 -> link_L4; limit lower=-3 upper=3 effort=10 velocity=3 -> lower=-2.55 upper=2.55 effort=14 velocity=6; parent link_L4 -> link_L3
- joint joint_J5: child link_L6 -> link_L5; limit lower=-3 upper=3 effort=10 velocity=3 -> lower=-2.55 upper=2.55 effort=14 velocity=6; parent link_L5 -> link_L4
- joint joint_J6: child link7 -> link_L6; limit lower=-3 upper=3 effort=10 velocity=3 -> lower=-2.92 upper=2.92 effort=14 velocity=6; parent link_L6 -> link_L5

Commit message: fix base orientation

File: motive_description/urdf/msa6_v03.urdf (robot description, URDF)
Before this commit: robot msa6, 8 links, 7 joints
Joints:
- joint joint_J1: origin xyz=0 0 0 rpy=0 0 -1.5708 -> xyz=0 0 0 rpy=0 0 0
