Commit message: Update EE rotation

File: motive_description/urdf/msa6_v03_on_stand.urdf.xacro (robot description, xacro)
@@ -18,5 +18,5 @@
     <parent link="link_L6" />
     <child link = "wrist_link" />
-    <origin xyz="0 0 0.05" rpy="${-pi/2} 0 ${pi/4}" />
+    <origin xyz="0 0 0.05" rpy="${-pi/2} 0 ${5*pi/8}" />
   </joint>
   <!-- end-effector -->

Commit message: Move the robot down to match reality

File: motive_description/urdf/msa6_v03_on_stand.urdf.xacro (robot description, xacro)
@@ -8,5 +8,5 @@
     <parent link="world" />
     <child link = "base_link" />
-    <origin xyz="0.194 0.369 1.73" rpy="1.5708 0 1.5708" />
+    <origin xyz="0.194 0.369 1.5875" rpy="1.5708 0 1.5708" />
   </joint>
   <link name="world" />
