Commit message: Remove the prefix on joints/links
...until a better solution can be found, Motive's software requires every robot arm to have consistent names

File: motive_description/urdf/msa6_v03.urdf.xacro (robot description, xacro)
@@ -15,5 +15,5 @@
     </link>
     <joint name="fixed" type="fixed">
-      <parent link="${prefix}base_link"/>
+      <parent link="base_link"/>
       <child link="link_L0"/>
       <!-- Floating to avoid collision-->
@@ -22,5 +22,5 @@
     </joint>
     <link
-      name="${prefix}link_L0">
+      name="link_L0">
       <inertial>
         <origin
@@ -62,5 +62,5 @@
     </link>
     <joint
-      name="${prefix}joint_J1"
+      name="joint_J1"
       type="revolute">
       <origin
@@ -84,5 +84,5 @@
     </joint>
     <link
-      name="${prefix}link_L1">
+      name="link_L1">
       <inertial>
         <origin
@@ -124,5 +124,5 @@
     </link>
     <joint
-      name="${prefix}joint_J2"
+      name="joint_J2"
       type="revolute">
       <origin
@@ -144,5 +144,5 @@
     </joint>
     <link
-      name="${prefix}link_L2">
+      name="link_L2">
       <inertial>
         <origin
@@ -184,5 +184,5 @@
     </link>
     <joint
-      name="${prefix}joint_J3"
+      name="joint_J3"
       type="revolute">
       <origin
@@ -204,5 +204,5 @@
     </joint>
     <link
-      name="${prefix}link_L3">
+      name="link_L3">
       <inertial>
         <origin
@@ -244,5 +244,5 @@
     </link>
     <joint
-      name="${prefix}joint_J4"
+      name="joint_J4"
       type="revolute">
       <origin
@@ -264,5 +264,5 @@
     </joint>
     <link
-      name="${prefix}link_L4">
+      name="link_L4">
       <inertial>
         <origin
@@ -304,5 +304,5 @@
     </link>
     <joint
-      name="${prefix}joint_J5"
+      name="joint_J5"
       type="revolute">
       <origin
@@ -324,5 +324,5 @@
     </joint>
     <link
-      name="${prefix}link_L5">
+      name="link_L5">
       <inertial>
         <origin
@@ -364,5 +364,5 @@
     </link>
     <joint
-      name="${prefix}joint_J6"
+      name="joint_J6"
       type="revolute">
       <origin
@@ -384,5 +384,5 @@
     </joint>
     <link
-      name="${prefix}link_L6">
+      name="link_L6">
       <inertial>
         <origin

Commit message: Incorporate 90deg base rotation. Restore prefixes

File: motive_description/urdf/msa6_v03.urdf.xacro (robot description, xacro)
@@ -16,5 +16,5 @@
     <joint name="fixed" type="fixed">
       <parent link="base_link"/>
-      <child link="link_L0"/>
+      <child link="${prefix}link_L0"/>
       <!-- Floating to avoid collision-->
       <origin
@@ -22,5 +22,5 @@
     </joint>
     <link
-      name="link_L0">
+      name="${prefix}link_L0">
       <inertial>
         <origin
@@ -62,13 +62,13 @@
     </link>
     <joint
-      name="joint_J1"
+      name="${prefix}joint_J1"
       type="revolute">
       <origin
         xyz="0 0 0"
-        rpy="0 0 -1.5708" />
-      <parent
-        link="link_L0" />
-      <child
-        link="link_L1" />
+        rpy="0 0 0" />
+      <parent
+        link="${prefix}link_L0" />
+      <child
+        link="${prefix}link_L1" />
       <axis
         xyz="0 0 1" />
@@ -84,5 +84,5 @@
     </joint>
     <link
-      name="link_L1">
+      name="${prefix}link_L1">
       <inertial>
         <origin
@@ -124,5 +124,5 @@
     </link>
     <joint
-      name="joint_J2"
+      name="${prefix}joint_J2"
       type="revolute">
       <origin
@@ -130,7 +130,7 @@
         rpy="0 1.5708 0" />
       <parent
-        link="link_L1" />
-      <child
-        link="link_L2" />
+        link="${prefix}link_L1" />
+      <child
+        link="${prefix}link_L2" />
       <axis
         xyz="0 0 1" />
@@ -144,5 +144,5 @@
     </joint>
     <link
-      name="link_L2">
+      name="${prefix}link_L2">
       <inertial>
         <origin
@@ -184,5 +184,5 @@
     </link>
     <joint
-      name="joint_J3"
+      name="${prefix}joint_J3"
       type="revolute">
       <origin
@@ -190,7 +190,7 @@
         rpy="3.1416 -1.5708 3.1416" />
       <parent
-        link="link_L2" />
-      <child
-        link="link_L3" />
+        link="${prefix}link_L2" />
+      <child
+        link="${prefix}link_L3" />
       <axis
         xyz="0 0 1" />
@@ -204,5 +204,5 @@
     </joint>
     <link
-      name="link_L3">
+      name="${prefix}link_L3">
       <inertial>
         <origin
@@ -244,5 +244,5 @@
     </link>
     <joint
-      name="joint_J4"
+      name="${prefix}joint_J4"
       type="revolute">
       <origin
@@ -250,7 +250,7 @@
         rpy="0 0 0" />
       <parent
-        link="link_L3" />
-      <child
-        link="link_L4" />
+        link="${prefix}link_L3" />
+      <child
+        link="${prefix}link_L4" />
       <axis
         xyz="0 0 1" />
@@ -264,5 +264,5 @@
     </joint>
     <link
-      name="link_L4">
+      name="${prefix}link_L4">
       <inertial>
         <origin
@@ -304,5 +304,5 @@
     </link>
     <joint
-      name="joint_J5"
+      name="${prefix}joint_J5"
       type="revolute">
       <origin
@@ -310,7 +310,7 @@
         rpy="-3.1416 0 3.1416" />
       <parent
-        link="link_L4" />
-      <child
-        link="link_L5" />
+        link="${prefix}link_L4" />
+      <child
+        link="${prefix}link_L5" />
       <axis
         xyz="0 0 1" />
@@ -324,5 +324,5 @@
     </joint>
     <link
-      name="link_L5">
+      name="${prefix}link_L5">
       <inertial>
         <origin
@@ -364,5 +364,5 @@
     </link>
     <joint
-      name="joint_J6"
+      name="${prefix}joint_J6"
       type="revolute">
       <origin
@@ -370,7 +370,7 @@
         rpy="-1.5708 -1.4987 1.5708" />
       <parent
-        link="link_L5" />
-      <child
-        link="link_L6" />
+        link="${prefix}link_L5" />
+      <child
+        link="${prefix}link_L6" />
       <axis
         xyz="0 0 1" />
@@ -384,5 +384,5 @@
     </joint>
     <link
-      name="link_L6">
+      name="${prefix}link_L6">
       <inertial>
         <origin

Commit message: Update joint names

File: motive_description/urdf/msa6_v03.urdf.xacro (robot description, xacro)
@@ -3,21 +3,10 @@
   xmlns:xacro="http://www.ros.org/wiki/xacro">
   <xacro:macro name="msa6" params="prefix">
-    <link name="${prefix}base_link">
-      <visual>
-        <geometry>
-          <box size="1.80 1.70 0.25"/>
-        </geometry>
-          <origin rpy="0 0 0.0" xyz="0.0 0 -0.125"/>
-    <material name="Gray">
-      <color rgba="0.8 0.8 0.8 1.0"/>
-    </material>
-      </visual>
-    </link>
+    <link name="${prefix}base_link" />
     <joint name="fixed" type="fixed">
       <parent link="base_link"/>
       <child link="${prefix}link_L0"/>
-      <!-- Floating to avoid collision-->
-      <origin
-        xyz="0 0 .15" />
+      <origin
+        xyz="0 0 0" />
     </joint>
     <link

Commit message: Remove the extra table description.
Don't make the arm floating anymore.

File: motive_description/urdf/msa6_v03.urdf.xacro (robot description, xacro)
@@ -3,21 +3,8 @@
   xmlns:xacro="http://www.ros.org/wiki/xacro">
   <xacro:macro name="msa6" params="prefix">
-    <link name="${prefix}base_link">
-      <visual>
-        <geometry>
-          <box size="1.80 1.70 0.25"/>
-        </geometry>
-          <origin rpy="0 0 0.0" xyz="0.0 0 -0.125"/>
-    <material name="Gray">
-      <color rgba="0.8 0.8 0.8 1.0"/>
-    </material>
-      </visual>
-    </link>
+    <link name="${prefix}base_link" />
     <joint name="fixed" type="fixed">
       <parent link="base_link"/>
       <child link="${prefix}link_L0"/>
-      <!-- Floating to avoid collision-->
-      <origin
-        xyz="0 0 .15" />
     </joint>
     <link

Commit message: update changes based on onsite adjustements

File: motive_description/urdf/msa6_v03.urdf.xacro (robot description, xacro)
@@ -7,4 +7,7 @@
       <parent link="base_link"/>
       <child link="${prefix}link_L0"/>
+      <origin
+          xyz="0 0 0.10795"
+          rpy="0 0 0" />
     </joint>
     <link

File: motive_description/urdf/msa6_v03_on_stand.urdf.xacro (robot description, xacro)
@@ -8,5 +8,5 @@
     <parent link="world" />
     <child link = "base_link" />
-    <origin xyz="0.194 0.369 1.5875" rpy="1.5708 0 1.5708" />
+    <origin xyz="0.06985 0.369 1.5275" rpy="1.5708 0 1.5708" />
   </joint>
   <link name="world" />
